File: PiZeroHub.sch (KiCad schematic (older format))
At the start: 28 parts, among them CON1 BARREL_JACK, P1 USB_OTG, P2 USB_OTG, P3 USB_B, P4 USB_B, P5 USB_B, P6 USB_B, P7 USB_OTG, U1 FE1_1_4PORTUSB, U2 LM7805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

Commit message: Finish first version
Parts:
- added C10, C11, C8, C9: 100uF, Capacitors_SMD:c_elec_5x5.3, symbol CP1_Small
- added F1: 1A, Fuse_Holders_and_Fuses:Fuse_SMD1206_Wave, symbol F_Small
- added F2: 1.5A, Fuse_Holders_and_Fuses:Fuse_SMD1206_Wave, symbol F_Small
Connections:
- net +5V: now also C10.1, C11.1, C8.1, C9.1, F1.2, F2.2; no longer C7.1, P7.1 (VCC), U2.2 (VO)
- net GND: now also R1.1, C10.2, C11.2, C8.2, C9.2
- net X-: now reaches U1.2 (XOUT), Y1.1
- net X+: now reaches U1.3 (XIN), Y1.2
- net at P2.1 (VCC): no longer R1.1
- new net: C7.1, F2.1, U2.2 (VO)
- new net: F1.1, P7.1 (VCC)
Other:
- moved on the sheet: R1

Commit message: latest version, new USB part and footprint, cleaner design
Parts:
- removed C6: 0.33uF, project_footprint:C_0402_Hand, symbol C_Small
- removed C7: 0.1uF, project_footprint:C_0402_Hand, symbol C_Small
- removed CON1: BARREL_JACK, Connect:BARREL_JACK, symbol BARREL_JACK
- removed F1: 1A, Fuse_Holders_and_Fuses:Fuse_SMD1206_Wave, symbol F_Small
- removed U2: LM7805, project_footprints:sot223, symbol LM7805
- added U2, U3, U4, U5: USBLC6-2, project_footprints:SOT-666, symbol USBLC6-2
- C1, C2, C4: Digikey Part No. (none) -> 399-3684-1-ND
- C10, C11, C8, C9: Digikey Part No. (none) -> PCE3853CT-ND
- C3, C5: Digikey Part No. (none) -> 587-1227-1-ND
- D1, D2, D3, D4: Digikey Part No. (none) -> 160-1446-1-ND
- D5: Digikey Part No. (none) -> 160-1447-1-ND
- F2: value 1.5A -> 2A; Digikey Part No. (none) -> SF-1206F150-2CT-ND
- P1, P2: Digikey Part No. (none) -> H11496CT-ND
- P3, P4, P5, P6: Digikey Part No. (none) -> ED2988-ND
- P7: value USB_OTG -> USB_POWER; Digikey Part No. (none) -> H11497-ND
- R1: Digikey Part No. (none) -> 311-100KLRCT-ND
- R2: Digikey Part No. (none) -> 311-2.7KJRCT-ND
- R3, R4, R5: Digikey Part No. (none) -> 311-1.00KLRCT-ND
- Y1: Digikey Part No. (none) -> 535-9100-1-ND
Connections:
- net +5V: now also U2.5 (VCC), U3.5 (VCC), U4.5 (VCC), U5.5 (VCC)
- net GND: now also U2.2 (GND), U3.2 (GND), U4.2 (GND), U5.2 (GND)
- net D1-: now reaches P3.2 (D-), U1.10 (D-1)
- net D1-: now also U2.1 (I/O_1), U2.6 (I/O_1)
- net D1+: now reaches P3.3 (D+), U1.11 (D+1)
- net D1+: now also U2.3 (I/O_2), U2.4 (I/O_2)
- net D4-: now reaches P6.2 (D-), U1.4 (D-4)
- net D4-: now also U5.1 (I/O_1), U5.6 (I/O_1)
- net D4+: now reaches P6.3 (D+), U1.5 (D+4)
- net D4+: now also U5.3 (I/O_2), U5.4 (I/O_2)
- net D3-: now reaches P5.2 (D-), U1.6 (D-3)
- net D3-: now also U4.3 (I/O_2), U4.4 (I/O_2)
- net D3+: now reaches P5.3 (D+), U1.7 (D+3)
- net D3+: now also U4.1 (I/O_1), U4.6 (I/O_1)
- net D2-: now reaches P4.2 (D-), U1.8 (D-2)
- net D2-: now also U3.3 (I/O_2), U3.4 (I/O_2)
- net D2+: now reaches P4.3 (D+), U1.9 (D+2)
- net D2+: now also U3.1 (I/O_1), U3.6 (I/O_1)
- net at F2.1: now also P7.1 (VCC)
Other:
- note added: "External Power 5V 2A\n\n"
- note removed: "External Power 6-15V\n"
- moved on the sheet: F2, P1
